File: board/power.kicad_sch (KiCad schematic)
At the start: 15 parts, among them IC1 MP4462DN-Z-LF, J1 MPM-15-24

Commit message: Traces, traces everywhere
Other:
- moved on the sheet: R12
Changed lines of the file:
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@@
   (junction (at 129.54 41.91) (diameter 0) (color 0 0 0 0)
   )
-  (junction (at 151.13 53.34) (diameter 0) (color 0 0 0 0)
-  )
   (junction (at 68.58 83.82) (diameter 0) (color 0 0 0 0)
   )
   (junction (at 100.33 53.34) (diameter 0) (color 0 0 0 0)
   )
+  (junction (at 105.41 49.53) (diameter 0) (color 0 0 0 0)
+  )
   (junction (at 97.79 49.53) (diameter 0) (color 0 0 0 0)
   )
@@
   (junction (at 35.56 44.45) (diameter 0) (color 0 0 0 0)
   )
-  (junction (at 129.54 53.34) (diameter 0) (color 0 0 0 0)
+  (junction (at 151.13 59.69) (diameter 0) (color 0 0 0 0)
   )
   (junction (at 95.25 49.53) (diameter 0) (color 0 0 0 0)
@@
     (stroke (width 0) (type default) (color 0 0 0 0))
   )
+  (wire (pts (xy 140.97 59.69) (xy 105.41 59.69))
+    (stroke (width 0) (type default) (color 0 0 0 0))
+  )
   (wire (pts (xy 63.5 83.82) (xy 68.58 83.82))
     (stroke (width 0) (type default) (color 0 0 0 0))
@@
     (stroke (width 0) (type default) (color 0 0 0 0))
   )
+  (wire (pts (xy 105.41 49.53) (xy 106.68 49.53))
+    (stroke (width 0) (type default) (color 0 0 0 0))
+  )
   (wire (pts (xy 71.12 62.23) (xy 100.33 62.23))
     (stroke (width 0) (type default) (color 0 0 0 0))
@@
     (stroke (width 0) (type default) (color 0 0 0 0))
   )
-  (wire (pts (xy 100.33 49.53) (xy 106.68 49.53))
+  (wire (pts (xy 100.33 49.53) (xy 105.41 49.53))
     (stroke (width 0) (type default) (color 0 0 0 0))
   )
@@
     (stroke (width 0) (type default) (color 0 0 0 0))
   )
-  (wire (pts (xy 151.13 73.66) (xy 151.13 53.34))
+  (wire (pts (xy 151.13 73.66) (xy 151.13 59.69))
     (stroke (width 0) (type default) (color 0 0 0 0))
   )
@@
     (stroke (width 0) (type default) (color 0 0 0 0))
   )
-  (wire (pts (xy 146.05 53.34) (xy 151.13 53.34))
+  (wire (pts (xy 146.05 59.69) (xy 151.13 59.69))
     (stroke (width 0) (type default) (color 0 0 0 0))
   )
@@
     (stroke (width 0) (type default) (color 0 0 0 0))
   )
+  (wire (pts (xy 151.13 49.53) (xy 151.13 59.69))
+    (stroke (width 0) (type default) (color 0 0 0 0))
+  )
   (wire (pts (xy 31.75 44.45) (xy 35.56 44.45))
     (stroke (width 0) (type default) (color 0 0 0 0))
@@
     (stroke (width 0) (type default) (color 0 0 0 0))
   )
-  (wire (pts (xy 151.13 53.34) (xy 151.13 49.53))
-    (stroke (width 0) (type default) (color 0 0 0 0))
-  )
   (wire (pts (xy 86.36 44.45) (xy 97.79 44.45))
     (stroke (width 0) (type default) (color 0 0 0 0))
@@
     (stroke (width 0) (type default) (color 0 0 0 0))
   )
-  (wire (pts (xy 129.54 53.34) (xy 140.97 53.34))
+  (wire (pts (xy 105.41 59.69) (xy 105.41 49.53))
     (stroke (width 0) (type default) (color 0 0 0 0))
   )
@@
     (pin "2")
   )
-  (symbol (lib_id "Device:R_Small") (at 143.51 53.34 270) (unit 1)
-    (in_bom yes) (on_board yes) (fields_autoplaced)
-    (property "Reference" "R12" (id 0) (at 143.51 46.99 90))
-    (property "Value" "40.2k" (id 1) (at 143.51 49.53 90))
-    (property "Footprint" "Resistor_SMD:R_0805_2012Metric" (id 2) (at 143.51 53.34 0)
-      (effects (font (size 1.27 1.27)) hide)
-    )
-    (property "Datasheet" "~" (id 3) (at 143.51 53.34 0)
-      (effects (font (size 1.27 1.27)) hide)
-    )
+  (symbol (lib_id "Device:R_Small") (at 143.51 59.69 270) (unit 1)
+    (in_bom yes) (on_board yes) (fields_autoplaced)
+    (property "Reference" "R12" (id 0) (at 143.51 53.34 90))
+    (property "Value" "40.2k" (id 1) (at 143.51 55.88 90))
+    (property "Footprint" "Resistor_SMD:R_0805_2012Metric" (id 2) (at 143.51 59.69 0)
+      (effects (font (size 1.27 1.27)) hide)
+    )
+    (property "Datasheet" "~" (id 3) (at 143.51 59.69 0)
+      (effects (font (size 1.27 1.27)) hide)
+    )

Commit message: RP2040 Stamp
Parts:
- removed C5: 22uF, Capacitor_SMD:C_0805_2012Metric, symbol Device:C_Small
- removed IC1: MP4462DN-Z-LF, SamacSys_Parts:SOIC127P600X170-9N, symbol SamacSys_Parts:MP4462DN-Z-LF
- removed R10: 100K, Resistor_SMD:R_0805_2012Metric, symbol Device:R_Small
- removed R11: 200k, Resistor_SMD:R_0805_2012Metric, symbol Device:R_Small
- removed R12: 40.2k, Resistor_SMD:R_0805_2012Metric, symbol Device:R_Small
- removed R13: 210k, Resistor_SMD:R_0805_2012Metric, symbol Device:R_Small
- added C5: 330uF, SamacSys_Parts:POSCAP_D12_D15_D15E_D2E_D2_D3L_D4, symbol Device:C_Polarized_Small
- added C6: 0.01uF, Capacitor_SMD:C_0805_2012Metric, symbol Device:C_Small
- added IC1: TPS5450DDA, SamacSys_Parts:SOIC127P600X170-9N, symbol SamacSys_Parts:TPS5450DDA
- C1: value 150pF -> 4.7uF
- C2: value NS -> 4.7uF
- C3: value 100nF -> 0.01uF
- C4: value 10uF -> 0.01uF
- D2: value B5819W SL -> B540C; footprint SamacSys_Parts:DIONM5127X229N -> SamacSys_Parts:DIOM7959X250N
- L1: value 22uH -> 15uH; footprint Inductor_SMD:L_12x12mm_H4.5mm -> SamacSys_Parts:INDPM120120X800N
- R7: value 17.4k -> 10k
- R8: value 100K -> 3.16k
Connections:
- net 24V: now also C1.1, C2.1, C3.1, IC1.7 (VIN); no longer C4.1, R7.2, R8.1
- net 5V: now also D2.1 (K), R7.2, C5.1, C6.1
- net GND: now also C1.2, C3.2, R8.1, C5.2, C6.2, IC1.6 (GND), IC1.9 (EP); no longer C4.2, R7.1
- net at R8.2: now also R7.1, IC1.4 (VSENSE)
- new net: C4.1, IC1.1 (BOOT)
- new net: C4.2, IC1.8 (PH), L1.1
- no-connect marks 0 -> 2

Commit message: Power shit and copper fillz boi
Connections:
- net 5Vunf: now reaches C4.2, IC1.8 (PH), L1.1
Changed lines of the file:
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@@
     (stroke (width 0) (type default) (color 0 0 0 0))
+  )
+  (label "5Vunf" (at 119.38 29.21 0)
+    (effects (font (size 1.27 1.27)) (justify left bottom))
   )
   (global_label "24V" (shape input) (at 25.4 29.21 180) (fields_autoplaced)

Commit message: TPs, vias, some comments on board, fml
Parts:
- added TP17: 5V, TestPoint:TestPoint_Pad_D1.5mm, symbol Connector:TestPoint_Small
- renumbered IC1 to IC3, J1 to J2, R7 to R10, R8 to R11
Connections:
- net 5V: now also TP17.1
Changed lines of the file:
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@@
   (junction (at 176.53 40.64) (diameter 0) (color 0 0 0 0)
+  )
+  (junction (at 184.15 29.21) (diameter 0) (color 0 0 0 0)
   )
   (junction (at 41.91 60.96) (diameter 0) (color 0 0 0 0)
@@
     (stroke (width 0) (type default) (color 0 0 0 0))
   )
-  (wire (pts (xy 176.53 29.21) (xy 190.5 29.21))
+  (wire (pts (xy 176.53 29.21) (xy 184.15 29.21))
+    (stroke (width 0) (type default) (color 0 0 0 0))
+  )
+  (wire (pts (xy 184.15 29.21) (xy 190.5 29.21))
     (stroke (width 0) (type default) (color 0 0 0 0))
   )
@@
     (stroke (width 0) (type default) (color 0 0 0 0))
   )
-  (wire (pts (xy 176.53 52.07) (xy 176.53 48.26))
+  (wire (pts (xy 176.53 48.26) (xy 176.53 52.07))
     (stroke (width 0) (type default) (color 0 0 0 0))
   )
@@
   (symbol (lib_id "SamacSys_Parts:MPM-15-24") (at 67.31 115.57 180) (unit 1)
     (in_bom yes) (on_board yes) (fields_autoplaced)
-    (property "Reference" "J1" (id 0) (at 54.61 105.41 0))
+    (property "Reference" "J2" (id 0) (at 54.61 105.41 0))
     (property "Value" "MPM-15-24" (id 1) (at 54.61 107.95 0))
     (property "Footprint" "SamacSys_Parts:MPM1524" (id 2) (at 45.72 118.11 0)
@@
     (pin "2")
   )
+  (symbol (lib_id "Connector:TestPoint_Small") (at 184.15 29.21 0) (unit 1)
+    (in_bom yes) (on_board yes) (fields_autoplaced)
+    (property "Reference" "TP17" (id 0) (at 185.42 27.9399 0)
+      (effects (font (size 1.27 1.27)) (justify left))
+    )
+    (property "Value" "5V" (id 1) (at 185.42 30.4799 0)
+      (effects (font (size 1.27 1.27)) (justify left))
+    )
+    (property "Footprint" "TestPoint:TestPoint_Pad_D1.5mm" (id 2) (at 189.23 29.21 0)
+      (effects (font (size 1.27 1.27)) hide)
+    )
+    (property "Datasheet" "~" (id 3) (at 189.23 29.21 0)
+      (effects (font (size 1.27 1.27)) hide)
+    )
+    (pin "1")
+  )
   (symbol (lib_id "Device:C_Polarized_Small") (at 148.59 34.29 0) (unit 1)
     (in_bom yes) (on_board yes) (fields_autoplaced)
@@
   (symbol (lib_id "Device:R_Small") (at 176.53 34.29 180) (unit 1)
     (in_bom yes) (on_board yes) (fields_autoplaced)
-    (property "Reference" "R7" (id 0) (at 179.07 33.0199 0)
+    (property "Reference" "R10" (id 0) (at 179.07 33.0199 0)
       (effects (font (size 1.27 1.27)) (justify right))
     )
@@
   (symbol (lib_id "SamacSys_Parts:TPS5450DDA") (at 72.39 29.21 0) (unit 1)
     (in_bom yes) (on_board yes) (fields_autoplaced)
-    (property "Reference" "IC1" (id 0) (at 87.63 21.59 0))
+    (property "Reference" "IC3" (id 0) (at 87.63 21.59 0))
     (property "Value" "TPS5450DDA" (id 1) (at 87.63 24.13 0))
     (property "Footprint" "SamacSys_Parts:SOIC127P600X170-9N" (id 2) (at 99.06 26.67 0)
@@
   (symbol (lib_id "Device:R_Small") (at 176.53 45.72 180) (unit 1)
     (in_bom yes) (on_board yes) (fields_autoplaced)
-    (property "Reference" "R8" (id 0) (at 179.07 44.4499 0)
+    (property "Reference" "R11" (id 0) (at 179.07 44.4499 0)
       (effects (font (size 1.27 1.27)) (justify right))
     )

Commit message: pushpushpush
Parts:
- removed C1, C2: 4.7uF, Capacitor_SMD:C_0805_2012Metric, symbol Device:C_Small
- removed C3, C4, C6: 0.01uF, Capacitor_SMD:C_0805_2012Metric, symbol Device:C_Small
- removed C5: 330uF, SamacSys_Parts:POSCAP_D12_D15_D15E_D2E_D2_D3L_D4, symbol Device:C_Polarized_Small
- removed D2: B540C, SamacSys_Parts:DIOM7959X250N, symbol Device:D_Schottky_Small
- removed IC3: TPS5450DDA, SamacSys_Parts:SOIC127P600X170-9N, symbol SamacSys_Parts:TPS5450DDA
- removed L1: 15uH, SamacSys_Parts:INDPM120120X800N, symbol Device:L_Small
- removed R10: 10k, Resistor_SMD:R_0805_2012Metric, symbol Device:R_Small
- removed R11: 3.16k, Resistor_SMD:R_0805_2012Metric, symbol Device:R_Small
- removed TP17: 5V, TestPoint:TestPoint_Pad_D1.5mm, symbol Connector:TestPoint_Small
- added JP1: RCON, Jumper:SolderJumper-2_P1.3mm_Open_RoundedPad1.0x1.5mm, symbol Jumper:SolderJumper_2_Bridged
- added PS2: SKMW20F-05, SamacSys_Parts:SKMW20F05, symbol SamacSys_Parts:SKMW20F-05
- added R1: TrimUP, Resistor_SMD:R_0805_2012Metric, symbol Device:R_Small
- added R2: TrimDOWN, Resistor_SMD:R_0805_2012Metric, symbol Device:R_Small
- added TP18: 5V, TestPoint:TestPoint_Pad_D1.5mm, symbol Connector:TestPoint_Small
- added TP2: RC, TestPoint:TestPoint_Pad_D1.5mm, symbol Connector:TestPoint_Small
- renumbered J2 to PS1
Connections:
- net 24V: now also JP1.1 (A), PS2.1 (+VIN)
- net 5V: now also PS2.3 (+VOUT), R2.2, TP18.1
- net GND: now also PS2.2 (-VIN), PS2.5 (-VOUT), R1.1
- new net: PS2.4 (TRIM), R1.2, R2.1
- new net: JP1.2 (B), PS2.6 (R.C.), TP2.1
- no-connect marks 2 -> 0
